Commit message: abstracted reward functions further; further tuning of standing and walking policies; new meshes + urdf; added reward for toe vs calf walking

File: source/rocket/rocket/data/Rocket.urdf (robot description, URDF)
Before this commit: robot Rocket, 7 links, 6 joints
Links:
- removed link Calf_Assy_L_1
- removed link Calf_Assy_R_1
- removed link Hip_Assy_L_1
- removed link Hip_Assy_R_1
- removed link Thigh_Assy_L_1
- removed link Thigh_Assy_R_1
- removed link Torso_Assy_1
- added link Calf_L_1, mass 0.106437; collision mesh filename=package://meshes/Calf_L_1.stl scale=0.001 0.001 0.001; visual mesh filename=package://meshes/Calf_L_1.stl scale=0.001 0.001 0.001
- added link Calf_R_1, mass 0.106436; collision mesh filename=package://meshes/Calf_R_1.stl scale=0.001 0.001 0.001; visual mesh filename=package://meshes/Calf_R_1.stl scale=0.001 0.001 0.001
- added link Hip_L_1, mass 1.017088; collision mesh filename=package://meshes/Hip_L_1.stl scale=0.001 0.001 0.001; visual mesh filename=package://meshes/Hip_L_1.stl scale=0.001 0.001 0.001
- added link Hip_R_1, mass 1.017208; collision mesh filename=package://meshes/Hip_R_1.stl scale=0.001 0.001 0.001; visual mesh filename=package://meshes/Hip_R_1.stl scale=0.001 0.001 0.001
- added link Thigh_L_1, mass 1.225024; collision mesh filename=package://meshes/Thigh_L_1.stl scale=0.001 0.001 0.001; visual mesh filename=package://meshes/Thigh_L_1.stl scale=0.001 0.001 0.001
- added link Thigh_R_1, mass 1.225024; collision mesh filename=package://meshes/Thigh_R_1.stl scale=0.001 0.001 0.001; visual mesh filename=package://meshes/Thigh_R_1.stl scale=0.001 0.001 0.001
- added link Toe_L_1, mass 0.015585; collision mesh filename=package://meshes/Toe_L_1.stl scale=0.001 0.001 0.001; visual mesh filename=package://meshes/Toe_L_1.stl scale=0.001 0.001 0.001
- added link Toe_R_1, mass 0.015585; collision mesh filename=package://meshes/Toe_R_1.stl scale=0.001 0.001 0.001; visual mesh filename=package://meshes/Toe_R_1.stl scale=0.001 0.001 0.001
- added link Torso_1, mass 1.658125; collision mesh filename=package://meshes/Torso_1.stl scale=0.001 0.001 0.001; visual mesh filename=package://meshes/Torso_1.stl scale=0.001 0.001 0.001
Joints:
- added joint Rigid7: type fixed, parent Calf_L_1, child Toe_L_1, origin xyz=-0.037 -0.087 -0.075 rpy=0 0 0
- added joint Rigid8: type fixed, parent Calf_R_1, child Toe_R_1, origin xyz=0.037 -0.087 -0.075 rpy=0 0 0
- joint Revolute1: axis 0 0 1 -> 0 0 -1; child Hip_Assy_L_1 -> Hip_L_1; limit lower=-0.2618 upper=0.2618 effort=1000 velocity=100 -> lower=-0.2618 upper=0.0872 effort=1000 velocity=100; origin xyz=-0.066 0 0.113 rpy=0 0 0 -> xyz=-0.066 0 0.02 rpy=0 0 0; parent Torso_Assy_1 -> Torso_1
- joint Revolute2: child Hip_Assy_R_1 -> Hip_R_1; limit lower=-0.2618 upper=0.2618 effort=1000 velocity=100 -> lower=-0.2618 upper=0.0872 effort=1000 velocity=100; origin xyz=0.066 0 0.113 rpy=0 0 0 -> xyz=0.066 0 0.02 rpy=0 0 0; parent Torso_Assy_1 -> Torso_1
- joint Revolute3: axis 1 0 0 -> 1.0 0.0 0.0; child Thigh_Assy_L_1 -> Thigh_L_1; limit lower=-0.1745 upper=0.1745 effort=1000 velocity=100 -> lower=-0.3490 upper=0.1745 effort=1000 velocity=100; origin xyz=-0.0491 0 -0.043 rpy=0 0 0 -> xyz=-0.049 0 0.05 rpy=0 0 0; parent Hip_Assy_L_1 -> Hip_L_1
- joint Revolute4: axis 1 0 0 -> 1.0 0.0 0.0; child Thigh_Assy_R_1 -> Thigh_R_1; limit lower=-0.1745 upper=0.1745 effort=1000 velocity=100 -> lower=-0.3490 upper=0.1745 effort=1000 velocity=100; origin xyz=0.0491 0 -0.043 rpy=0 0 0 -> xyz=0.049 0 0.05 rpy=0 0 0; parent Hip_Assy_R_1 -> Hip_R_1
- joint Revolute5: axis -1 0 0 -> -1.0 0 0; child Calf_Assy_L_1 -> Calf_L_1; limit lower=-0.1745 upper=0.1745 effort=1000 velocity=100 -> lower=-0.3490 upper=0.2618 effort=1000 velocity=100; origin xyz=-0.0488 0.099 -0.099 rpy=0 0 0 -> xyz=0.014 0.099 -0.099 rpy=0 0 0; parent Thigh_Assy_L_1 -> Thigh_L_1
- joint Revolute6: axis -1 0 0 -> -1.0 0 0; child Calf_Assy_R_1 -> Calf_R_1; limit lower=-0.1745 upper=0.1745 effort=1000 velocity=100 -> lower=-0.3490 upper=0.2618 effort=1000 velocity=100; origin xyz=0.0488 0.099 -0.099 rpy=0 0 0 -> xyz=-0.014 0.099 -0.099 rpy=0 0 0; parent Thigh_Assy_R_1 -> Thigh_R_1

Commit message: made mass randomization better esp. for torso electronics

File: source/rocket/rocket/data/Rocket.urdf (robot description, URDF)
Before this commit: robot RocketForURDF, 9 links, 8 joints
Links:
- link Torso_1: mass 1.658125 -> 2.358125

Commit message: new policyyy

File: source/rocket/rocket/data/Rocket.urdf (robot description, URDF)
Before this commit: robot RocketForURDF, 9 links, 8 joints
Links:
- link Torso_1: mass 2.358125 -> 2.158125

Commit message: jumping penalty + loer hip limits

File: source/rocket/rocket/data/Rocket.urdf (robot description, URDF)
Before this commit: robot RocketForURDF, 9 links, 8 joints
Joints:
- joint Revolute1: limit lower=-0.2618 upper=0.0872 effort=1000 velocity=100 -> lower=-0.0349 upper=0.0349 effort=1000 velocity=100
- joint Revolute2: limit lower=-0.2618 upper=0.0872 effort=1000 velocity=100 -> lower=-0.0349 upper=0.0349 effort=1000 velocity=100

Commit message: made standing not step; reduced effort and joint limits for knees

File: source/rocket/rocket/data/Rocket.urdf (robot description, URDF)
Before this commit: robot RocketForURDF, 9 links, 8 joints
Joints:
- joint Revolute5: limit lower=-0.3490 upper=0.2618 effort=1000 velocity=100 -> lower=-0.3490 upper=0.1 effort=1000 velocity=100
- joint Revolute6: limit lower=-0.3490 upper=0.2618 effort=1000 velocity=100 -> lower=-0.3490 upper=0.1 effort=1000 velocity=100

Commit message: upped effort joint limits

File: source/rocket/rocket/data/Rocket.urdf (robot description, URDF)
Before this commit: robot RocketForURDF, 9 links, 8 joints
Joints:
- joint Revolute5: limit lower=-0.3490 upper=0.1 effort=1000 velocity=100 -> lower=-0.3490 upper=0.2618 effort=1000 velocity=100
- joint Revolute6: limit lower=-0.3490 upper=0.1 effort=1000 velocity=100 -> lower=-0.3490 upper=0.2618 effort=1000 velocity=100

Commit message: limit joints more

File: source/rocket/rocket/data/Rocket.urdf (robot description, URDF)
Before this commit: robot RocketForURDF, 9 links, 8 joints
Joints:
- joint Revolute3: limit lower=-0.3490 upper=0.1745 effort=1000 velocity=100 -> lower=-0.2618 upper=0.1745 effort=1000 velocity=100
- joint Revolute4: limit lower=-0.3490 upper=0.1745 effort=1000 velocity=100 -> lower=-0.2618 upper=0.1745 effort=1000 velocity=100
- joint Revolute5: limit lower=-0.3490 upper=0.2618 effort=1000 velocity=100 -> lower=-0.3490 upper=0.0873 effort=1000 velocity=100
- joint Revolute6: limit lower=-0.3490 upper=0.2618 effort=1000 velocity=100 -> lower=-0.3490 upper=0.0873 effort=1000 velocity=100

Commit message: old joint limits

File: source/rocket/rocket/data/Rocket.urdf (robot description, URDF)
Before this commit: robot RocketForURDF, 9 links, 8 joints
Joints:
- joint Revolute3: limit lower=-0.2618 upper=0.1745 effort=1000 velocity=100 -> lower=-0.3490 upper=0.1745 effort=1000 velocity=100
- joint Revolute4: limit lower=-0.2618 upper=0.1745 effort=1000 velocity=100 -> lower=-0.3490 upper=0.1745 effort=1000 velocity=100
- joint Revolute5: limit lower=-0.3490 upper=0.0873 effort=1000 velocity=100 -> lower=-0.3490 upper=0.2618 effort=1000 velocity=100
- joint Revolute6: limit lower=-0.3490 upper=0.0873 effort=1000 velocity=100 -> lower=-0.3490 upper=0.2618 effort=1000 velocity=100
